File: projects/touch-panel/work3/_rip2.kicad_pcb (KiCad board)
At the start: 2 copper layers, 71 x 150 mm, 269 parts, among them J1 FPC-40P-0.5mm, Q1 AO3400, Q10 AO3400, Q100 AO3400, Q101 AO3400, Q102 AO3400, Q103 AO3400, Q104 AO3400, Q105 AO3400, Q106 AO3400, Q107 AO3400, Q108 AO3400, Q109 AO3400, Q11 AO3400, Q110 AO3400, Q111 AO3400, Q112 AO3400, Q113 AO3400, Q114 AO3400, Q115 AO3400, Q116 AO3400, Q117 AO3400, Q118 AO3400, Q119 AO3400, Q12 AO3400, Q120 AO3400, Q121 AO3400, Q122 AO3400, Q123 AO3400, Q124 AO3400, Q125 AO3400, Q126 AO3400, Q127 AO3400, Q128 AO3400, Q129 AO3400, Q13 AO3400, Q130 AO3400, Q131 AO3400, Q132 AO3400, Q133 AO3400, Q134 AO3400, Q135 AO3400, Q136 AO3400, Q137 AO3400, Q138 AO3400, Q139 AO3400, Q14 AO3400, Q140 AO3400, Q141 AO3400, Q142 AO3400, Q143 AO3400, Q144 AO3400, Q145 AO3400, Q146 AO3400, Q147 AO3400, Q148 AO3400, Q149 AO3400, Q15 AO3400, Q150 AO3400, Q151 AO3400, Q152 AO3400, Q153 AO3400, Q154 AO3400, Q155 AO3400, Q156 AO3400, Q157 AO3400, Q158 AO3400, Q159 AO3400, Q16 AO3400, Q160 AO3400, Q161 AO3400, Q162 AO3400, Q163 AO3400, Q164 AO3400, Q165 AO3400, Q166 AO3400, Q167 AO3400, Q168 AO3400, Q169 AO3400, Q17 AO3400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

Commit message: touch-panel完成work3
Parts:
- removed J1: FPC-40P-0.5mm, Connector_FFC-FPC:Hirose_FH12-40S-0.5SH_1x40-1MP_P0.50mm_Horizontal
- added J1A: PinHeader_1x20_P2.54mm_Vertical, PinHeader_1x20_P2.54mm_Vertical, F.Cu at (95.4, 115.7)
- added J1B: PinHeader_1x20_P2.54mm_Vertical, PinHeader_1x20_P2.54mm_Vertical, F.Cu at (175.6, 181.0)
Routing:
- net GND: track 325.4 -> 147.4 mm
- net CSEL3: track 255.8 -> 120.7 mm, vias 5 -> 4
- net CSEL4: track 234.7 -> 101.7 mm, vias 5 -> 3
- net ROW1: track 223.2 -> 92.4 mm, vias 2 -> 1
- net CSEL5: track 216.1 -> 88.8 mm
- net ROW0: track 256.9 -> 135.7 mm, vias 10 -> 9
- net CSEL6: track 191.3 -> 70.1 mm
- net ROW2: track 211.9 -> 90.9 mm, vias 4 -> 0
- net ROW4: track 236.0 -> 127.7 mm
- net ROW6: track 212.7 -> 114.3 mm, vias 2 -> 1
- net ROW7: track 204.7 -> 116.9 mm, vias 2 -> 1
- net ROW8: track 173.9 -> 91.6 mm, vias 2 -> 1
- net ROW9: track 185.5 -> 117.7 mm, vias 4 -> 2
- net ROW10: track 194.0 -> 126.4 mm, vias 4 -> 3
- net ROW11: track 193.7 -> 126.8 mm, vias 4 -> 3
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Other:
- board size 71 x 150 mm -> 91 x 150 mm
