File: projects/touch-panel/work3/_spur.kicad_pcb (KiCad board)
At the start: 2 copper layers, 71 x 150 mm, 269 parts, among them J1 FPC-40P-0.5mm, Q1 AO3400, Q10 AO3400, Q100 AO3400, Q101 AO3400, Q102 AO3400, Q103 AO3400, Q104 AO3400, Q105 AO3400, Q106 AO3400, Q107 AO3400, Q108 AO3400, Q109 AO3400, Q11 AO3400, Q110 AO3400, Q111 AO3400, Q112 AO3400, Q113 AO3400, Q114 AO3400, Q115 AO3400, Q116 AO3400, Q117 AO3400, Q118 AO3400, Q119 AO3400, Q12 AO3400, Q120 AO3400, Q121 AO3400, Q122 AO3400, Q123 AO3400, Q124 AO3400, Q125 AO3400, Q126 AO3400, Q127 AO3400, Q128 AO3400, Q129 AO3400, Q13 AO3400, Q130 AO3400, Q131 AO3400, Q132 AO3400, Q133 AO3400, Q134 AO3400, Q135 AO3400, Q136 AO3400, Q137 AO3400, Q138 AO3400, Q139 AO3400, Q14 AO3400, Q140 AO3400, Q141 AO3400, Q142 AO3400, Q143 AO3400, Q144 AO3400, Q145 AO3400, Q146 AO3400, Q147 AO3400, Q148 AO3400, Q149 AO3400, Q15 AO3400, Q150 AO3400, Q151 AO3400, Q152 AO3400, Q153 AO3400, Q154 AO3400, Q155 AO3400, Q156 AO3400, Q157 AO3400, Q158 AO3400, Q159 AO3400, Q16 AO3400, Q160 AO3400, Q161 AO3400, Q162 AO3400, Q163 AO3400, Q164 AO3400, Q165 AO3400, Q166 AO3400, Q167 AO3400, Q168 AO3400, Q169 AO3400, Q17 AO3400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

Commit message: touch-panel完成work3
Parts:
- added J1A: PinHeader_1x20_P2.54mm_Vertical, PinHeader_1x20_P2.54mm_Vertical, F.Cu at (95.4, 115.7)
- added J1B: PinHeader_1x20_P2.54mm_Vertical, PinHeader_1x20_P2.54mm_Vertical, F.Cu at (175.6, 181.0)
Routing:
- net CSEL3: track 255.8 -> 0.00 mm, vias 5 -> 0
- net CSEL4: track 234.7 -> 0.00 mm, vias 5 -> 0
- net ROW4: track 236.0 -> 66.8 mm, vias 4 -> 0
- net ROW1: track 223.2 -> 62.7 mm, vias 2 -> 0
- net ROW6: track 212.7 -> 68.1 mm, vias 2 -> 0
- net ROW7: track 204.7 -> 68.6 mm, vias 2 -> 0
- net ROW10: track 194.0 -> 63.3 mm, vias 4 -> 0
- net ROW11: track 193.7 -> 79.7 mm, vias 4 -> 0
- net ROW9: track 185.5 -> 77.7 mm, vias 4 -> 1
- net ROW12: track 152.6 -> 57.6 mm, vias 2 -> 0
- net ROW13: track 155.9 -> 63.2 mm, vias 2 -> 0
- net GND: track 325.4 -> 273.5 mm, vias 2 -> 0
- net ROW18: track 129.7 -> 83.9 mm, vias 4 -> 2
- net CSEL5: track 216.1 -> 179.0 mm, vias 3 -> 1
- net CSEL0: track 35.0 -> 4.52 mm, vias 4 -> 0
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Other:
- board size 71 x 150 mm -> 91 x 150 mm
