File: projects/touch-panel/work3/_t3.kicad_pcb (KiCad board)
At the start: 2 copper layers, 71 x 150 mm, 269 parts, among them J1 FPC-40P-0.5mm, Q1 AO3400, Q10 AO3400, Q100 AO3400, Q101 AO3400, Q102 AO3400, Q103 AO3400, Q104 AO3400, Q105 AO3400, Q106 AO3400, Q107 AO3400, Q108 AO3400, Q109 AO3400, Q11 AO3400, Q110 AO3400, Q111 AO3400, Q112 AO3400, Q113 AO3400, Q114 AO3400, Q115 AO3400, Q116 AO3400, Q117 AO3400, Q118 AO3400, Q119 AO3400, Q12 AO3400, Q120 AO3400, Q121 AO3400, Q122 AO3400, Q123 AO3400, Q124 AO3400, Q125 AO3400, Q126 AO3400, Q127 AO3400, Q128 AO3400, Q129 AO3400, Q13 AO3400, Q130 AO3400, Q131 AO3400, Q132 AO3400, Q133 AO3400, Q134 AO3400, Q135 AO3400, Q136 AO3400, Q137 AO3400, Q138 AO3400, Q139 AO3400, Q14 AO3400, Q140 AO3400, Q141 AO3400, Q142 AO3400, Q143 AO3400, Q144 AO3400, Q145 AO3400, Q146 AO3400, Q147 AO3400, Q148 AO3400, Q149 AO3400, Q15 AO3400, Q150 AO3400, Q151 AO3400, Q152 AO3400, Q153 AO3400, Q154 AO3400, Q155 AO3400, Q156 AO3400, Q157 AO3400, Q158 AO3400, Q159 AO3400, Q16 AO3400, Q160 AO3400, Q161 AO3400, Q162 AO3400, Q163 AO3400, Q164 AO3400, Q165 AO3400, Q166 AO3400, Q167 AO3400, Q168 AO3400, Q169 AO3400, Q17 AO3400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

Commit message: touch-panel完成work3
Parts:
- removed J1: FPC-40P-0.5mm, Connector_FFC-FPC:Hirose_FH12-40S-0.5SH_1x40-1MP_P0.50mm_Horizontal
- added J1A: PinHeader_1x20_P2.54mm_Vertical, PinHeader_1x20_P2.54mm_Vertical, F.Cu at (95.4, 115.7)
- added J1B: PinHeader_1x20_P2.54mm_Vertical, PinHeader_1x20_P2.54mm_Vertical, F.Cu at (175.6, 181.0)
Routing:
- net CSEL2: track 26.7 -> 154.5 mm, vias 2 -> 5
- net CSEL1: track 28.5 -> 153.6 mm, vias 2 -> 6
- net CSEL0: track 35.0 -> 158.7 mm, vias 4 -> 6
- net ROW19: track 78.9 -> 196.9 mm, vias 2 -> 6
- net ROW15: track 136.8 -> 252.6 mm, vias 2 -> 4
- net ROW10: track 194.0 -> 83.8 mm, vias 4 -> 2
- net ROW2: track 211.9 -> 102.7 mm, vias 4 -> 1
- net ROW20: track 74.8 -> 182.2 mm, vias 2 -> 6
- net CSEL6: track 191.3 -> 296.3 mm, vias 4 -> 11
- net ROW11: track 193.7 -> 92.3 mm, vias 4 -> 0
- net ROW14: track 177.3 -> 269.0 mm, vias 4 -> 5
- net ROW17: track 90.4 -> 180.8 mm, vias 0 -> 1
- net ROW12: track 152.6 -> 77.4 mm, vias 2 -> 0
- net CSEL5: track 216.1 -> 142.3 mm, vias 3 -> 1
- net ROW9: track 185.5 -> 114.0 mm, vias 4 -> 5
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Other:
- board size 71 x 150 mm -> 91 x 150 mm
