File: projects/touch-panel/work3/replan/p5.kicad_pcb (KiCad board)
At the start: 2 copper layers, 71 x 150 mm, 269 parts, among them J1 FPC-40P-0.5mm, Q1 AO3400, Q10 AO3400, Q100 AO3400, Q101 AO3400, Q102 AO3400, Q103 AO3400, Q104 AO3400, Q105 AO3400, Q106 AO3400, Q107 AO3400, Q108 AO3400, Q109 AO3400, Q11 AO3400, Q110 AO3400, Q111 AO3400, Q112 AO3400, Q113 AO3400, Q114 AO3400, Q115 AO3400, Q116 AO3400, Q117 AO3400, Q118 AO3400, Q119 AO3400, Q12 AO3400, Q120 AO3400, Q121 AO3400, Q122 AO3400, Q123 AO3400, Q124 AO3400, Q125 AO3400, Q126 AO3400, Q127 AO3400, Q128 AO3400, Q129 AO3400, Q13 AO3400, Q130 AO3400, Q131 AO3400, Q132 AO3400, Q133 AO3400, Q134 AO3400, Q135 AO3400, Q136 AO3400, Q137 AO3400, Q138 AO3400, Q139 AO3400, Q14 AO3400, Q140 AO3400, Q141 AO3400, Q142 AO3400, Q143 AO3400, Q144 AO3400, Q145 AO3400, Q146 AO3400, Q147 AO3400, Q148 AO3400, Q149 AO3400, Q15 AO3400, Q150 AO3400, Q151 AO3400, Q152 AO3400, Q153 AO3400, Q154 AO3400, Q155 AO3400, Q156 AO3400, Q157 AO3400, Q158 AO3400, Q159 AO3400, Q16 AO3400, Q160 AO3400, Q161 AO3400, Q162 AO3400, Q163 AO3400, Q164 AO3400, Q165 AO3400, Q166 AO3400, Q167 AO3400, Q168 AO3400, Q169 AO3400, Q17 AO3400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

Commit message: touch-panel完成work3
Routing:
- net COL4: track 193.8 -> 30.6 mm, vias 22 -> 4
- net ROW12: track 152.6 -> 34.1 mm, vias 2 -> 1
- net ROW3: track 62.8 -> 177.7 mm
- net ROW16: track 122.9 -> 35.3 mm, vias 2 -> 0
- net ROW5: track 62.7 -> 133.8 mm
- net ROW8: track 173.9 -> 113.9 mm, vias 2 -> 0
- net ROW14: track 177.3 -> 119.8 mm, vias 4 -> 2
- net ROW7: track 204.7 -> 255.4 mm, vias 2 -> 1
- net ROW17: track 90.4 -> 50.7 mm
- net ROW19: track 78.9 -> 42.5 mm, vias 2 -> 1
- net ROW6: track 212.7 -> 176.4 mm
- net ROW9: track 185.5 -> 152.1 mm
- net ROW11: track 193.7 -> 161.9 mm, vias 4 -> 3
- net ROW18: track 129.7 -> 98.2 mm, vias 4 -> 3
- net ROW4: track 236.0 -> 205.0 mm
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